File: techin514_final/techin514_final.kicad_sch (KiCad schematic)
At the start: 6 parts, among them SW1 SW_Push_Dual_x2, U1 TSSP58038, U2 ESP32-C3

Commit message: Updates
Parts:
- removed D1: LED_ARBG, symbol Device:LED_ARBG
- removed U1: TSSP58038, OptoDevice:Vishay_MINICAST-3Pin, symbol Sensor_Proximity:TSSP58038
- removed U2: ESP32-C3, Package_DFN_QFN:QFN-32-1EP_5x5mm_P0.5mm_EP3.7x3.7mm, symbol MCU_Espressif:ESP32-C3
- added D1: SFH4546, LED_THT:LED_D5.0mm_IRGrey, symbol LED:SFH4546
- added EXP32_c3: ~, RF_Module:MCU_Seeed_ESP32C3, symbol Shareef 32:XIAO_ESP32_SENSE
- added R2: 10K, Resistor_THT:R_Axial_DIN0204_L3.6mm_D1.6mm_P1.90mm_Vertical, symbol Device:R
- added R3: 10k, Resistor_THT:R_Axial_DIN0204_L3.6mm_D1.6mm_P1.90mm_Vertical, symbol Device:R
- added SW2: SW_Push_Dual_x2, Button_Switch_THT:SW_XKB_DM1-16UC-1, symbol Switch:SW_Push_Dual_x2
- added U2: HC‑SR501 Sensor Board, OptoDevice:Vishay_MINICAST-3Pin, symbol Sensor_Proximity:TSSP58038
- R1: value R -> 220 Ω; footprint (none) -> Resistor_THT:R_Axial_DIN0204_L3.6mm_D1.6mm_P1.90mm_Vertical
- SW1: footprint (none) -> Button_Switch_THT:SW_PUSH_6mm_H4.3mm
Connections:
- net at R1.1: now also EXP32_c3.3 (GPIO3_A2_D2)
- net at BT1.1 (+): now also EXP32_c3.8 (5V), U2.3 (Vs); no longer R1.2
- net at BT1.2 (-), SW1.2 (D): now also D1.1 (K), SW2.2 (D), U2.2 (GND)
- net at SW1.1 (C): now also EXP32_c3.4 (GPIO4_A3_D3), R2.1
- new net: D1.2 (A), R1.2
- new net: EXP32_c3.2 (GPIO2_A1_D1), U2.1 (OUT)
- new net: EXP32_c3.10 (3V3), R2.2, R3.2
- new net: EXP32_c3.5 (GPIO4_A3_D3_SDA), R3.1, SW2.1 (C)
- no-connect marks 0 -> 1
Other:
- company: (none) -> GIX-MSTI
- title: (none) -> Shoppers Sensors
- moved on the sheet: SW1A
